Commit message: live selector with slider now works, replaced module stls with cylinders

File: urdf/actuator.xacro (robot description, xacro)
@@ -76,8 +76,16 @@
     <link name="${name}/INPUT_INTERFACE">
       <visual>
-        <origin xyz="0 0 0" rpy="0 0 0" />
-        <geometry>
-          <mesh filename="${mesh_filename}" scale="0.001 0.001 0.001"/>
-        </geometry>
+        <xacro:if value="${model_name.startswith('X5')}">
+          <origin xyz="0 0 0.0125" rpy="0 0 0" />
+          <geometry>
+            <cylinder radius="0.035" length="0.025"/>
+          </geometry>
+        </xacro:if>
+        <xacro:if value="${model_name.startswith('X8')}">
+          <origin xyz="0 0 0.02" rpy="0 0 0" />
+          <geometry>
+            <cylinder radius="0.035" length="0.04"/>
+          </geometry>
+        </xacro:if>
         <xacro:unless value="${model_name.startswith('R8')}">
           <xacro:red_material/>
@@ -88,8 +96,16 @@
       </visual>
       <collision>
-        <origin xyz="0 0 0" rpy="0 0 0" />
-        <geometry>
-          <mesh filename="${mesh_filename}" scale="0.001 0.001 0.001"/>
-        </geometry>
+        <xacro:if value="${model_name.startswith('X5')}">
+          <origin xyz="0 0 0.0125" rpy="0 0 0" />
+          <geometry>
+            <cylinder radius="0.035" length="0.025"/>
+          </geometry>
+        </xacro:if>
+        <xacro:if value="${model_name.startswith('X8')}">
+          <origin xyz="0 0 0.02" rpy="0 0 0" />
+          <geometry>
+            <cylinder radius="0.035" length="0.04"/>
+          </geometry>
+        </xacro:if>
       </collision>
       <inertial>
@@ -117,12 +133,4 @@
       </inertial>
     </link>
-    <gazebo reference="${name}/INPUT_INTERFACE">
-      <xacro:unless value="${model_name.startswith('R8')}">
-        <xacro:gazebo_red_material/>
-      </xacro:unless>
-      <xacro:if value="${model_name.startswith('R8')}">
-        <xacro:gazebo_black_material/>
-      </xacro:if>
-    </gazebo>
     <joint name="${name}/${model_name}" type="${urdf_joint_type}">
       <parent link="${name}/INPUT_INTERFACE"/>

File: urdf/bracket.xacro (robot description, xacro)
@@ -150,12 +150,4 @@
     </xacro:if>
   </link>
-  <gazebo reference="${name}/INPUT_INTERFACE">
-    <xacro:if value="${bracket_type.startswith('X5Light') or bracket_type.startswith('R5Light')}">
-      <xacro:gazebo_beige_material/>
-    </xacro:if>
-    <xacro:if value="${bracket_type.startswith('X5Heavy') or bracket_type.startswith('R5Heavy')}">
-      <xacro:gazebo_black_material/>
-    </xacro:if>
-  </gazebo>
   <joint name="${name}/OUTPUT_INTERFACE" type="fixed">
     <parent link="${name}/INPUT_INTERFACE"/>
@@ -180,8 +172,4 @@
     </xacro:if>
   </joint>
-  <gazebo reference="${name}/OUTPUT_INTERFACE">
-    <disableFixedJointLumping>true</disableFixedJointLumping>
-    <preserveFixedJoint>true</preserveFixedJoint>
-  </gazebo>
   </xacro:macro>
 </robot>

File: urdf/hebi.xacro (robot description, xacro)
@@ -45,7 +45,7 @@
   <!-- <xacro:include filename="end_effector.xacro"/> -->
   <!-- This automatically loads the gazebo plugin for xacro models
-       which include hebi.xacro -->
+       which include hebi.xacro
   <gazebo>
     <plugin name="hebi_gazebo_plugin" filename="libhebi_gazebo_plugin.so"/>
-  </gazebo>
+  </gazebo>-->
 </robot>

File: urdf/leg.xacro (robot description, xacro)
@@ -22,5 +22,5 @@
     <visual>
       <geometry>
-        <sphere radius="0.025"/>
+        <sphere radius="0.02"/>
       </geometry>
             <origin xyz="0 0 -.02" rpy="0 0 0"/>
@@ -29,12 +29,9 @@
   <collision>
         <geometry>
-          <sphere radius="0.025"/>
+          <sphere radius="0.02"/>
         </geometry>
                   <origin xyz="0 0 -.02" rpy="0 0 0"/>
   </collision>
   </link>
-<!--
-  <xacro:null_end_effector name="leg_${num}/J3_elbow"/>
--->
   <!-- use rubber bit for foot end link; necessary to provide output for HEBI components to attach to. -->
   </xacro:macro>

File: urdf/link.xacro (robot description, xacro)
@@ -52,7 +52,4 @@
       </inertial>
     </link>
-    <gazebo reference="${name}/INPUT_INTERFACE">
-      <xacro:gazebo_silver_material/>
-    </gazebo>
     <joint name="${name}/OUTPUT_JOINT" type="fixed">
       <parent link="${name}/INPUT_INTERFACE"/>
@@ -60,8 +57,4 @@
       <origin xyz="${extension} ${-sin(twist) * edge_to_center} ${edge_to_center * (1 + cos(twist))}" rpy="${twist} 0 0"/>
     </joint>
-    <gazebo reference="${name}/OUTPUT_JOINT">
-      <disableFixedJointLumping>true</disableFixedJointLumping>
-      <preserveFixedJoint>true</preserveFixedJoint>
-    </gazebo>
   </xacro:macro>
 </robot>

File: urdf/llllll.urdf (robot description, URDF)
Before this commit: robot llllll, 43 links, 42 joints
Links:
- link leg_1/J1_base/INPUT_INTERFACE: geometry collision cylinder length=0.04 radius=0.035; visual cylinder length=0.04 radius=0.035
- link leg_1/J2_shoulder/INPUT_INTERFACE: geometry collision cylinder length=0.04 radius=0.035; visual cylinder length=0.04 radius=0.035
- link leg_1/J3_elbow/INPUT_INTERFACE: geometry collision cylinder length=0.025 radius=0.035; visual cylinder length=0.025 radius=0.035
- link leg_1/foot/INPUT_INTERFACE: geometry collision sphere radius=0.02; visual sphere radius=0.02
- link leg_2/J1_base/INPUT_INTERFACE: geometry collision cylinder length=0.04 radius=0.035; visual cylinder length=0.04 radius=0.035
- link leg_2/J2_shoulder/INPUT_INTERFACE: geometry collision cylinder length=0.04 radius=0.035; visual cylinder length=0.04 radius=0.035
- link leg_2/J3_elbow/INPUT_INTERFACE: geometry collision cylinder length=0.025 radius=0.035; visual cylinder length=0.025 radius=0.035
- link leg_2/foot/INPUT_INTERFACE: geometry collision sphere radius=0.02; visual sphere radius=0.02
- link leg_3/J1_base/INPUT_INTERFACE: geometry collision cylinder length=0.04 radius=0.035; visual cylinder length=0.04 radius=0.035
- link leg_3/J2_shoulder/INPUT_INTERFACE: geometry collision cylinder length=0.04 radius=0.035; visual cylinder length=0.04 radius=0.035
- link leg_3/J3_elbow/INPUT_INTERFACE: geometry collision cylinder length=0.025 radius=0.035; visual cylinder length=0.025 radius=0.035
- link leg_3/foot/INPUT_INTERFACE: geometry collision sphere radius=0.02; visual sphere radius=0.02
- link leg_4/J1_base/INPUT_INTERFACE: geometry collision cylinder length=0.04 radius=0.035; visual cylinder length=0.04 radius=0.035
- link leg_4/J2_shoulder/INPUT_INTERFACE: geometry collision cylinder length=0.04 radius=0.035; visual cylinder length=0.04 radius=0.035
- link leg_4/J3_elbow/INPUT_INTERFACE: geometry collision cylinder length=0.025 radius=0.035; visual cylinder length=0.025 radius=0.035
- link leg_4/foot/INPUT_INTERFACE: geometry collision sphere radius=0.02; visual sphere radius=0.02
- link leg_5/J1_base/INPUT_INTERFACE: geometry collision cylinder length=0.04 radius=0.035; visual cylinder length=0.04 radius=0.035
- link leg_5/J2_shoulder/INPUT_INTERFACE: geometry collision cylinder length=0.04 radius=0.035; visual cylinder length=0.04 radius=0.035
- link leg_5/J3_elbow/INPUT_INTERFACE: geometry collision cylinder length=0.025 radius=0.035; visual cylinder length=0.025 radius=0.035
- link leg_5/foot/INPUT_INTERFACE: geometry collision sphere radius=0.02; visual sphere radius=0.02
- link leg_6/J1_base/INPUT_INTERFACE: geometry collision cylinder length=0.04 radius=0.035; visual cylinder length=0.04 radius=0.035
- link leg_6/J2_shoulder/INPUT_INTERFACE: geometry collision cylinder length=0.04 radius=0.035; visual cylinder length=0.04 radius=0.035
- link leg_6/J3_elbow/INPUT_INTERFACE: geometry collision cylinder length=0.025 radius=0.035; visual cylinder length=0.025 radius=0.035
- link leg_6/foot/INPUT_INTERFACE: geometry collision sphere radius=0.02; visual sphere radius=0.02

File: urdf/llwwll.urdf (robot description, URDF)
Before this commit: robot llwwll, 37 links, 36 joints
Links:
- link leg_1/J1_base/INPUT_INTERFACE: geometry collision cylinder length=0.04 radius=0.035; visual cylinder length=0.04 radius=0.035
- link leg_1/J2_shoulder/INPUT_INTERFACE: geometry collision cylinder length=0.04 radius=0.035; visual cylinder length=0.04 radius=0.035
- link leg_1/J3_elbow/INPUT_INTERFACE: geometry collision cylinder length=0.025 radius=0.035; visual cylinder length=0.025 radius=0.035
- link leg_1/foot/INPUT_INTERFACE: geometry collision sphere radius=0.02; visual sphere radius=0.02
- link leg_2/J1_base/INPUT_INTERFACE: geometry collision cylinder length=0.04 radius=0.035; visual cylinder length=0.04 radius=0.035
- link leg_2/J2_shoulder/INPUT_INTERFACE: geometry collision cylinder length=0.04 radius=0.035; visual cylinder length=0.04 radius=0.035
- link leg_2/J3_elbow/INPUT_INTERFACE: geometry collision cylinder length=0.025 radius=0.035; visual cylinder length=0.025 radius=0.035
- link leg_2/foot/INPUT_INTERFACE: geometry collision sphere radius=0.02; visual sphere radius=0.02
- link leg_5/J1_base/INPUT_INTERFACE: geometry collision cylinder length=0.04 radius=0.035; visual cylinder length=0.04 radius=0.035
- link leg_5/J2_shoulder/INPUT_INTERFACE: geometry collision cylinder length=0.04 radius=0.035; visual cylinder length=0.04 radius=0.035
- link leg_5/J3_elbow/INPUT_INTERFACE: geometry collision cylinder length=0.025 radius=0.035; visual cylinder length=0.025 radius=0.035
- link leg_5/foot/INPUT_INTERFACE: geometry collision sphere radius=0.02; visual sphere radius=0.02
- link leg_6/J1_base/INPUT_INTERFACE: geometry collision cylinder length=0.04 radius=0.035; visual cylinder length=0.04 radius=0.035
- link leg_6/J2_shoulder/INPUT_INTERFACE: geometry collision cylinder length=0.04 radius=0.035; visual cylinder length=0.04 radius=0.035
- link leg_6/J3_elbow/INPUT_INTERFACE: geometry collision cylinder length=0.025 radius=0.035; visual cylinder length=0.025 radius=0.035
- link leg_6/foot/INPUT_INTERFACE: geometry collision sphere radius=0.02; visual sphere radius=0.02
- link wheel_3/J1_base/INPUT_INTERFACE: geometry collision cylinder length=0.025 radius=0.035; visual cylinder length=0.025 radius=0.035
- link wheel_3/J2_shoulder/INPUT_INTERFACE: geometry collision cylinder length=0.04 radius=0.035; visual cylinder length=0.04 radius=0.035
- link wheel_3/wheel/INPUT_INTERFACE: geometry collision cylinder length=0.0254 radius=0.105; visual cylinder length=0.0254 radius=0.105
- link wheel_4/J1_base/INPUT_INTERFACE: geometry collision cylinder length=0.025 radius=0.035; visual cylinder length=0.025 radius=0.035
- link wheel_4/J2_shoulder/INPUT_INTERFACE: geometry collision cylinder length=0.04 radius=0.035; visual cylinder length=0.04 radius=0.035
- link wheel_4/wheel/INPUT_INTERFACE: geometry collision cylinder length=0.0254 radius=0.105; visual cylinder length=0.0254 radius=0.105

File: urdf/lnllnl.urdf (robot description, URDF)
Before this commit: robot lnllnl, 29 links, 28 joints
Links:
- link leg_1/J1_base/INPUT_INTERFACE: geometry collision cylinder length=0.04 radius=0.035; visual cylinder length=0.04 radius=0.035
- link leg_1/J2_shoulder/INPUT_INTERFACE: geometry collision cylinder length=0.04 radius=0.035; visual cylinder length=0.04 radius=0.035
- link leg_1/J3_elbow/INPUT_INTERFACE: geometry collision cylinder length=0.025 radius=0.035; visual cylinder length=0.025 radius=0.035
- link leg_1/foot/INPUT_INTERFACE: geometry collision sphere radius=0.02; visual sphere radius=0.02
- link leg_3/J1_base/INPUT_INTERFACE: geometry collision cylinder length=0.04 radius=0.035; visual cylinder length=0.04 radius=0.035
- link leg_3/J2_shoulder/INPUT_INTERFACE: geometry collision cylinder length=0.04 radius=0.035; visual cylinder length=0.04 radius=0.035
- link leg_3/J3_elbow/INPUT_INTERFACE: geometry collision cylinder length=0.025 radius=0.035; visual cylinder length=0.025 radius=0.035
- link leg_3/foot/INPUT_INTERFACE: geometry collision sphere radius=0.02; visual sphere radius=0.02
- link leg_4/J1_base/INPUT_INTERFACE: geometry collision cylinder length=0.04 radius=0.035; visual cylinder length=0.04 radius=0.035
- link leg_4/J2_shoulder/INPUT_INTERFACE: geometry collision cylinder length=0.04 radius=0.035; visual cylinder length=0.04 radius=0.035
- link leg_4/J3_elbow/INPUT_INTERFACE: geometry collision cylinder length=0.025 radius=0.035; visual cylinder length=0.025 radius=0.035
- link leg_4/foot/INPUT_INTERFACE: geometry collision sphere radius=0.02; visual sphere radius=0.02
- link leg_6/J1_base/INPUT_INTERFACE: geometry collision cylinder length=0.04 radius=0.035; visual cylinder length=0.04 radius=0.035
- link leg_6/J2_shoulder/INPUT_INTERFACE: geometry collision cylinder length=0.04 radius=0.035; visual cylinder length=0.04 radius=0.035
- link leg_6/J3_elbow/INPUT_INTERFACE: geometry collision cylinder length=0.025 radius=0.035; visual cylinder length=0.025 radius=0.035
- link leg_6/foot/INPUT_INTERFACE: geometry collision sphere radius=0.02; visual sphere radius=0.02

File: urdf/lnwwnl.urdf (robot description, URDF)
Before this commit: robot lnwwnl, 23 links, 22 joints
Links:
- link leg_1/J1_base/INPUT_INTERFACE: geometry collision cylinder length=0.04 radius=0.035; visual cylinder length=0.04 radius=0.035
- link leg_1/J2_shoulder/INPUT_INTERFACE: geometry collision cylinder length=0.04 radius=0.035; visual cylinder length=0.04 radius=0.035
- link leg_1/J3_elbow/INPUT_INTERFACE: geometry collision cylinder length=0.025 radius=0.035; visual cylinder length=0.025 radius=0.035
- link leg_1/foot/INPUT_INTERFACE: geometry collision sphere radius=0.02; visual sphere radius=0.02
- link leg_6/J1_base/INPUT_INTERFACE: geometry collision cylinder length=0.04 radius=0.035; visual cylinder length=0.04 radius=0.035
- link leg_6/J2_shoulder/INPUT_INTERFACE: geometry collision cylinder length=0.04 radius=0.035; visual cylinder length=0.04 radius=0.035
- link leg_6/J3_elbow/INPUT_INTERFACE: geometry collision cylinder length=0.025 radius=0.035; visual cylinder length=0.025 radius=0.035
- link leg_6/foot/INPUT_INTERFACE: geometry collision sphere radius=0.02; visual sphere radius=0.02
- link wheel_3/J1_base/INPUT_INTERFACE: geometry collision cylinder length=0.025 radius=0.035; visual cylinder length=0.025 radius=0.035
- link wheel_3/J2_shoulder/INPUT_INTERFACE: geometry collision cylinder length=0.04 radius=0.035; visual cylinder length=0.04 radius=0.035
- link wheel_3/wheel/INPUT_INTERFACE: geometry collision cylinder length=0.0254 radius=0.105; visual cylinder length=0.0254 radius=0.105
- link wheel_4/J1_base/INPUT_INTERFACE: geometry collision cylinder length=0.025 radius=0.035; visual cylinder length=0.025 radius=0.035
- link wheel_4/J2_shoulder/INPUT_INTERFACE: geometry collision cylinder length=0.04 radius=0.035; visual cylinder length=0.04 radius=0.035
- link wheel_4/wheel/INPUT_INTERFACE: geometry collision cylinder length=0.0254 radius=0.105; visual cylinder length=0.0254 radius=0.105

File: urdf/lwllwl.urdf (robot description, URDF)
Before this commit: robot lwllwl, 37 links, 36 joints
Links:
- link leg_1/J1_base/INPUT_INTERFACE: geometry collision cylinder length=0.04 radius=0.035; visual cylinder length=0.04 radius=0.035
- link leg_1/J2_shoulder/INPUT_INTERFACE: geometry collision cylinder length=0.04 radius=0.035; visual cylinder length=0.04 radius=0.035
- link leg_1/J3_elbow/INPUT_INTERFACE: geometry collision cylinder length=0.025 radius=0.035; visual cylinder length=0.025 radius=0.035
- link leg_1/foot/INPUT_INTERFACE: geometry collision sphere radius=0.02; visual sphere radius=0.02
- link leg_3/J1_base/INPUT_INTERFACE: geometry collision cylinder length=0.04 radius=0.035; visual cylinder length=0.04 radius=0.035
- link leg_3/J2_shoulder/INPUT_INTERFACE: geometry collision cylinder length=0.04 radius=0.035; visual cylinder length=0.04 radius=0.035
- link leg_3/J3_elbow/INPUT_INTERFACE: geometry collision cylinder length=0.025 radius=0.035; visual cylinder length=0.025 radius=0.035
- link leg_3/foot/INPUT_INTERFACE: geometry collision sphere radius=0.02; visual sphere radius=0.02
- link leg_4/J1_base/INPUT_INTERFACE: geometry collision cylinder length=0.04 radius=0.035; visual cylinder length=0.04 radius=0.035
- link leg_4/J2_shoulder/INPUT_INTERFACE: geometry collision cylinder length=0.04 radius=0.035; visual cylinder length=0.04 radius=0.035
- link leg_4/J3_elbow/INPUT_INTERFACE: geometry collision cylinder length=0.025 radius=0.035; visual cylinder length=0.025 radius=0.035
- link leg_4/foot/INPUT_INTERFACE: geometry collision sphere radius=0.02; visual sphere radius=0.02
- link leg_6/J1_base/INPUT_INTERFACE: geometry collision cylinder length=0.04 radius=0.035; visual cylinder length=0.04 radius=0.035
- link leg_6/J2_shoulder/INPUT_INTERFACE: geometry collision cylinder length=0.04 radius=0.035; visual cylinder length=0.04 radius=0.035
- link leg_6/J3_elbow/INPUT_INTERFACE: geometry collision cylinder length=0.025 radius=0.035; visual cylinder length=0.025 radius=0.035
- link leg_6/foot/INPUT_INTERFACE: geometry collision sphere radius=0.02; visual sphere radius=0.02
- link wheel_2/J1_base/INPUT_INTERFACE: geometry collision cylinder length=0.025 radius=0.035; visual cylinder length=0.025 radius=0.035
- link wheel_2/J2_shoulder/INPUT_INTERFACE: geometry collision cylinder length=0.04 radius=0.035; visual cylinder length=0.04 radius=0.035
- link wheel_2/wheel/INPUT_INTERFACE: geometry collision cylinder length=0.0254 radius=0.105; visual cylinder length=0.0254 radius=0.105
- link wheel_5/J1_base/INPUT_INTERFACE: geometry collision cylinder length=0.025 radius=0.035; visual cylinder length=0.025 radius=0.035
- link wheel_5/J2_shoulder/INPUT_INTERFACE: geometry collision cylinder length=0.04 radius=0.035; visual cylinder length=0.04 radius=0.035
- link wheel_5/wheel/INPUT_INTERFACE: geometry collision cylinder length=0.0254 radius=0.105; visual cylinder length=0.0254 radius=0.105

File: urdf/lwwwwl.urdf (robot description, URDF)
Before this commit: robot lwwwwl, 31 links, 30 joints
Links:
- link leg_1/J1_base/INPUT_INTERFACE: geometry collision cylinder length=0.04 radius=0.035; visual cylinder length=0.04 radius=0.035
- link leg_1/J2_shoulder/INPUT_INTERFACE: geometry collision cylinder length=0.04 radius=0.035; visual cylinder length=0.04 radius=0.035
- link leg_1/J3_elbow/INPUT_INTERFACE: geometry collision cylinder length=0.025 radius=0.035; visual cylinder length=0.025 radius=0.035
- link leg_1/foot/INPUT_INTERFACE: geometry collision sphere radius=0.02; visual sphere radius=0.02
- link leg_6/J1_base/INPUT_INTERFACE: geometry collision cylinder length=0.04 radius=0.035; visual cylinder length=0.04 radius=0.035
- link leg_6/J2_shoulder/INPUT_INTERFACE: geometry collision cylinder length=0.04 radius=0.035; visual cylinder length=0.04 radius=0.035
- link leg_6/J3_elbow/INPUT_INTERFACE: geometry collision cylinder length=0.025 radius=0.035; visual cylinder length=0.025 radius=0.035
- link leg_6/foot/INPUT_INTERFACE: geometry collision sphere radius=0.02; visual sphere radius=0.02
- link wheel_2/J1_base/INPUT_INTERFACE: geometry collision cylinder length=0.025 radius=0.035; visual cylinder length=0.025 radius=0.035
- link wheel_2/J2_shoulder/INPUT_INTERFACE: geometry collision cylinder length=0.04 radius=0.035; visual cylinder length=0.04 radius=0.035
- link wheel_2/wheel/INPUT_INTERFACE: geometry collision cylinder length=0.0254 radius=0.105; visual cylinder length=0.0254 radius=0.105
- link wheel_3/J1_base/INPUT_INTERFACE: geometry collision cylinder length=0.025 radius=0.035; visual cylinder length=0.025 radius=0.035
- link wheel_3/J2_shoulder/INPUT_INTERFACE: geometry collision cylinder length=0.04 radius=0.035; visual cylinder length=0.04 radius=0.035
- link wheel_3/wheel/INPUT_INTERFACE: geometry collision cylinder length=0.0254 radius=0.105; visual cylinder length=0.0254 radius=0.105
- link wheel_4/J1_base/INPUT_INTERFACE: geometry collision cylinder length=0.025 radius=0.035; visual cylinder length=0.025 radius=0.035
- link wheel_4/J2_shoulder/INPUT_INTERFACE: geometry collision cylinder length=0.04 radius=0.035; visual cylinder length=0.04 radius=0.035
- link wheel_4/wheel/INPUT_INTERFACE: geometry collision cylinder length=0.0254 radius=0.105; visual cylinder length=0.0254 radius=0.105
- link wheel_5/J1_base/INPUT_INTERFACE: geometry collision cylinder length=0.025 radius=0.035; visual cylinder length=0.025 radius=0.035
- link wheel_5/J2_shoulder/INPUT_INTERFACE: geometry collision cylinder length=0.04 radius=0.035; visual cylinder length=0.04 radius=0.035
- link wheel_5/wheel/INPUT_INTERFACE: geometry collision cylinder length=0.0254 radius=0.105; visual cylinder length=0.0254 radius=0.105
