Commit message: live selector with slider now works, replaced module stls with cylinders

File: urdf/wllllw.urdf (robot description, URDF)
Before this commit: robot wllllw, 37 links, 36 joints
Links:
- link leg_2/J1_base/INPUT_INTERFACE: geometry collision cylinder length=0.04 radius=0.035; visual cylinder length=0.04 radius=0.035
- link leg_2/J2_shoulder/INPUT_INTERFACE: geometry collision cylinder length=0.04 radius=0.035; visual cylinder length=0.04 radius=0.035
- link leg_2/J3_elbow/INPUT_INTERFACE: geometry collision cylinder length=0.025 radius=0.035; visual cylinder length=0.025 radius=0.035
- link leg_2/foot/INPUT_INTERFACE: geometry collision sphere radius=0.02; visual sphere radius=0.02
- link leg_3/J1_base/INPUT_INTERFACE: geometry collision cylinder length=0.04 radius=0.035; visual cylinder length=0.04 radius=0.035
- link leg_3/J2_shoulder/INPUT_INTERFACE: geometry collision cylinder length=0.04 radius=0.035; visual cylinder length=0.04 radius=0.035
- link leg_3/J3_elbow/INPUT_INTERFACE: geometry collision cylinder length=0.025 radius=0.035; visual cylinder length=0.025 radius=0.035
- link leg_3/foot/INPUT_INTERFACE: geometry collision sphere radius=0.02; visual sphere radius=0.02
- link leg_4/J1_base/INPUT_INTERFACE: geometry collision cylinder length=0.04 radius=0.035; visual cylinder length=0.04 radius=0.035
- link leg_4/J2_shoulder/INPUT_INTERFACE: geometry collision cylinder length=0.04 radius=0.035; visual cylinder length=0.04 radius=0.035
- link leg_4/J3_elbow/INPUT_INTERFACE: geometry collision cylinder length=0.025 radius=0.035; visual cylinder length=0.025 radius=0.035
- link leg_4/foot/INPUT_INTERFACE: geometry collision sphere radius=0.02; visual sphere radius=0.02
- link leg_5/J1_base/INPUT_INTERFACE: geometry collision cylinder length=0.04 radius=0.035; visual cylinder length=0.04 radius=0.035
- link leg_5/J2_shoulder/INPUT_INTERFACE: geometry collision cylinder length=0.04 radius=0.035; visual cylinder length=0.04 radius=0.035
- link leg_5/J3_elbow/INPUT_INTERFACE: geometry collision cylinder length=0.025 radius=0.035; visual cylinder length=0.025 radius=0.035
- link leg_5/foot/INPUT_INTERFACE: geometry collision sphere radius=0.02; visual sphere radius=0.02
- link wheel_1/J1_base/INPUT_INTERFACE: geometry collision cylinder length=0.025 radius=0.035; visual cylinder length=0.025 radius=0.035
- link wheel_1/J2_shoulder/INPUT_INTERFACE: geometry collision cylinder length=0.04 radius=0.035; visual cylinder length=0.04 radius=0.035
- link wheel_1/wheel/INPUT_INTERFACE: geometry collision cylinder length=0.0254 radius=0.105; visual cylinder length=0.0254 radius=0.105
- link wheel_6/J1_base/INPUT_INTERFACE: geometry collision cylinder length=0.025 radius=0.035; visual cylinder length=0.025 radius=0.035
- link wheel_6/J2_shoulder/INPUT_INTERFACE: geometry collision cylinder length=0.04 radius=0.035; visual cylinder length=0.04 radius=0.035
- link wheel_6/wheel/INPUT_INTERFACE: geometry collision cylinder length=0.0254 radius=0.105; visual cylinder length=0.0254 radius=0.105

File: urdf/wlwwlw.urdf (robot description, URDF)
Before this commit: robot wlwwlw, 31 links, 30 joints
Links:
- link leg_2/J1_base/INPUT_INTERFACE: geometry collision cylinder length=0.04 radius=0.035; visual cylinder length=0.04 radius=0.035
- link leg_2/J2_shoulder/INPUT_INTERFACE: geometry collision cylinder length=0.04 radius=0.035; visual cylinder length=0.04 radius=0.035
- link leg_2/J3_elbow/INPUT_INTERFACE: geometry collision cylinder length=0.025 radius=0.035; visual cylinder length=0.025 radius=0.035
- link leg_2/foot/INPUT_INTERFACE: geometry collision sphere radius=0.02; visual sphere radius=0.02
- link leg_5/J1_base/INPUT_INTERFACE: geometry collision cylinder length=0.04 radius=0.035; visual cylinder length=0.04 radius=0.035
- link leg_5/J2_shoulder/INPUT_INTERFACE: geometry collision cylinder length=0.04 radius=0.035; visual cylinder length=0.04 radius=0.035
- link leg_5/J3_elbow/INPUT_INTERFACE: geometry collision cylinder length=0.025 radius=0.035; visual cylinder length=0.025 radius=0.035
- link leg_5/foot/INPUT_INTERFACE: geometry collision sphere radius=0.02; visual sphere radius=0.02
- link wheel_1/J1_base/INPUT_INTERFACE: geometry collision cylinder length=0.025 radius=0.035; visual cylinder length=0.025 radius=0.035
- link wheel_1/J2_shoulder/INPUT_INTERFACE: geometry collision cylinder length=0.04 radius=0.035; visual cylinder length=0.04 radius=0.035
- link wheel_1/wheel/INPUT_INTERFACE: geometry collision cylinder length=0.0254 radius=0.105; visual cylinder length=0.0254 radius=0.105
- link wheel_3/J1_base/INPUT_INTERFACE: geometry collision cylinder length=0.025 radius=0.035; visual cylinder length=0.025 radius=0.035
- link wheel_3/J2_shoulder/INPUT_INTERFACE: geometry collision cylinder length=0.04 radius=0.035; visual cylinder length=0.04 radius=0.035
- link wheel_3/wheel/INPUT_INTERFACE: geometry collision cylinder length=0.0254 radius=0.105; visual cylinder length=0.0254 radius=0.105
- link wheel_4/J1_base/INPUT_INTERFACE: geometry collision cylinder length=0.025 radius=0.035; visual cylinder length=0.025 radius=0.035
- link wheel_4/J2_shoulder/INPUT_INTERFACE: geometry collision cylinder length=0.04 radius=0.035; visual cylinder length=0.04 radius=0.035
- link wheel_4/wheel/INPUT_INTERFACE: geometry collision cylinder length=0.0254 radius=0.105; visual cylinder length=0.0254 radius=0.105
- link wheel_6/J1_base/INPUT_INTERFACE: geometry collision cylinder length=0.025 radius=0.035; visual cylinder length=0.025 radius=0.035
- link wheel_6/J2_shoulder/INPUT_INTERFACE: geometry collision cylinder length=0.04 radius=0.035; visual cylinder length=0.04 radius=0.035
- link wheel_6/wheel/INPUT_INTERFACE: geometry collision cylinder length=0.0254 radius=0.105; visual cylinder length=0.0254 radius=0.105

File: urdf/wnllnw.urdf (robot description, URDF)
Before this commit: robot wnllnw, 23 links, 22 joints
Links:
- link leg_3/J1_base/INPUT_INTERFACE: geometry collision cylinder length=0.04 radius=0.035; visual cylinder length=0.04 radius=0.035
- link leg_3/J2_shoulder/INPUT_INTERFACE: geometry collision cylinder length=0.04 radius=0.035; visual cylinder length=0.04 radius=0.035
- link leg_3/J3_elbow/INPUT_INTERFACE: geometry collision cylinder length=0.025 radius=0.035; visual cylinder length=0.025 radius=0.035
- link leg_3/foot/INPUT_INTERFACE: geometry collision sphere radius=0.02; visual sphere radius=0.02
- link leg_4/J1_base/INPUT_INTERFACE: geometry collision cylinder length=0.04 radius=0.035; visual cylinder length=0.04 radius=0.035
- link leg_4/J2_shoulder/INPUT_INTERFACE: geometry collision cylinder length=0.04 radius=0.035; visual cylinder length=0.04 radius=0.035
- link leg_4/J3_elbow/INPUT_INTERFACE: geometry collision cylinder length=0.025 radius=0.035; visual cylinder length=0.025 radius=0.035
- link leg_4/foot/INPUT_INTERFACE: geometry collision sphere radius=0.02; visual sphere radius=0.02
- link wheel_1/J1_base/INPUT_INTERFACE: geometry collision cylinder length=0.025 radius=0.035; visual cylinder length=0.025 radius=0.035
- link wheel_1/J2_shoulder/INPUT_INTERFACE: geometry collision cylinder length=0.04 radius=0.035; visual cylinder length=0.04 radius=0.035
- link wheel_1/wheel/INPUT_INTERFACE: geometry collision cylinder length=0.0254 radius=0.105; visual cylinder length=0.0254 radius=0.105
- link wheel_6/J1_base/INPUT_INTERFACE: geometry collision cylinder length=0.025 radius=0.035; visual cylinder length=0.025 radius=0.035
- link wheel_6/J2_shoulder/INPUT_INTERFACE: geometry collision cylinder length=0.04 radius=0.035; visual cylinder length=0.04 radius=0.035
- link wheel_6/wheel/INPUT_INTERFACE: geometry collision cylinder length=0.0254 radius=0.105; visual cylinder length=0.0254 radius=0.105

File: urdf/wnwwnw.urdf (robot description, URDF)
Before this commit: robot wnwwnw, 17 links, 16 joints
Links:
- link wheel_1/J1_base/INPUT_INTERFACE: geometry collision cylinder length=0.025 radius=0.035; visual cylinder length=0.025 radius=0.035
- link wheel_1/J2_shoulder/INPUT_INTERFACE: geometry collision cylinder length=0.04 radius=0.035; visual cylinder length=0.04 radius=0.035
- link wheel_1/wheel/INPUT_INTERFACE: geometry collision cylinder length=0.0254 radius=0.105; visual cylinder length=0.0254 radius=0.105
- link wheel_3/J1_base/INPUT_INTERFACE: geometry collision cylinder length=0.025 radius=0.035; visual cylinder length=0.025 radius=0.035
- link wheel_3/J2_shoulder/INPUT_INTERFACE: geometry collision cylinder length=0.04 radius=0.035; visual cylinder length=0.04 radius=0.035
- link wheel_3/wheel/INPUT_INTERFACE: geometry collision cylinder length=0.0254 radius=0.105; visual cylinder length=0.0254 radius=0.105
- link wheel_4/J1_base/INPUT_INTERFACE: geometry collision cylinder length=0.025 radius=0.035; visual cylinder length=0.025 radius=0.035
- link wheel_4/J2_shoulder/INPUT_INTERFACE: geometry collision cylinder length=0.04 radius=0.035; visual cylinder length=0.04 radius=0.035
- link wheel_4/wheel/INPUT_INTERFACE: geometry collision cylinder length=0.0254 radius=0.105; visual cylinder length=0.0254 radius=0.105
- link wheel_6/J1_base/INPUT_INTERFACE: geometry collision cylinder length=0.025 radius=0.035; visual cylinder length=0.025 radius=0.035
- link wheel_6/J2_shoulder/INPUT_INTERFACE: geometry collision cylinder length=0.04 radius=0.035; visual cylinder length=0.04 radius=0.035
- link wheel_6/wheel/INPUT_INTERFACE: geometry collision cylinder length=0.0254 radius=0.105; visual cylinder length=0.0254 radius=0.105

File: urdf/wwllww.urdf (robot description, URDF)
Before this commit: robot wwllww, 31 links, 30 joints
Links:
- link leg_3/J1_base/INPUT_INTERFACE: geometry collision cylinder length=0.04 radius=0.035; visual cylinder length=0.04 radius=0.035
- link leg_3/J2_shoulder/INPUT_INTERFACE: geometry collision cylinder length=0.04 radius=0.035; visual cylinder length=0.04 radius=0.035
- link leg_3/J3_elbow/INPUT_INTERFACE: geometry collision cylinder length=0.025 radius=0.035; visual cylinder length=0.025 radius=0.035
- link leg_3/foot/INPUT_INTERFACE: geometry collision sphere radius=0.02; visual sphere radius=0.02
- link leg_4/J1_base/INPUT_INTERFACE: geometry collision cylinder length=0.04 radius=0.035; visual cylinder length=0.04 radius=0.035
- link leg_4/J2_shoulder/INPUT_INTERFACE: geometry collision cylinder length=0.04 radius=0.035; visual cylinder length=0.04 radius=0.035
- link leg_4/J3_elbow/INPUT_INTERFACE: geometry collision cylinder length=0.025 radius=0.035; visual cylinder length=0.025 radius=0.035
- link leg_4/foot/INPUT_INTERFACE: geometry collision sphere radius=0.02; visual sphere radius=0.02
- link wheel_1/J1_base/INPUT_INTERFACE: geometry collision cylinder length=0.025 radius=0.035; visual cylinder length=0.025 radius=0.035
- link wheel_1/J2_shoulder/INPUT_INTERFACE: geometry collision cylinder length=0.04 radius=0.035; visual cylinder length=0.04 radius=0.035
- link wheel_1/wheel/INPUT_INTERFACE: geometry collision cylinder length=0.0254 radius=0.105; visual cylinder length=0.0254 radius=0.105
- link wheel_2/J1_base/INPUT_INTERFACE: geometry collision cylinder length=0.025 radius=0.035; visual cylinder length=0.025 radius=0.035
- link wheel_2/J2_shoulder/INPUT_INTERFACE: geometry collision cylinder length=0.04 radius=0.035; visual cylinder length=0.04 radius=0.035
- link wheel_2/wheel/INPUT_INTERFACE: geometry collision cylinder length=0.0254 radius=0.105; visual cylinder length=0.0254 radius=0.105
- link wheel_5/J1_base/INPUT_INTERFACE: geometry collision cylinder length=0.025 radius=0.035; visual cylinder length=0.025 radius=0.035
- link wheel_5/J2_shoulder/INPUT_INTERFACE: geometry collision cylinder length=0.04 radius=0.035; visual cylinder length=0.04 radius=0.035
- link wheel_5/wheel/INPUT_INTERFACE: geometry collision cylinder length=0.0254 radius=0.105; visual cylinder length=0.0254 radius=0.105
- link wheel_6/J1_base/INPUT_INTERFACE: geometry collision cylinder length=0.025 radius=0.035; visual cylinder length=0.025 radius=0.035
- link wheel_6/J2_shoulder/INPUT_INTERFACE: geometry collision cylinder length=0.04 radius=0.035; visual cylinder length=0.04 radius=0.035
- link wheel_6/wheel/INPUT_INTERFACE: geometry collision cylinder length=0.0254 radius=0.105; visual cylinder length=0.0254 radius=0.105

File: urdf/wwwwww.urdf (robot description, URDF)
Before this commit: robot wwwwww, 25 links, 24 joints
Links:
- link wheel_1/J1_base/INPUT_INTERFACE: geometry collision cylinder length=0.025 radius=0.035; visual cylinder length=0.025 radius=0.035
- link wheel_1/J2_shoulder/INPUT_INTERFACE: geometry collision cylinder length=0.04 radius=0.035; visual cylinder length=0.04 radius=0.035
- link wheel_1/wheel/INPUT_INTERFACE: geometry collision cylinder length=0.0254 radius=0.105; visual cylinder length=0.0254 radius=0.105
- link wheel_2/J1_base/INPUT_INTERFACE: geometry collision cylinder length=0.025 radius=0.035; visual cylinder length=0.025 radius=0.035
- link wheel_2/J2_shoulder/INPUT_INTERFACE: geometry collision cylinder length=0.04 radius=0.035; visual cylinder length=0.04 radius=0.035
- link wheel_2/wheel/INPUT_INTERFACE: geometry collision cylinder length=0.0254 radius=0.105; visual cylinder length=0.0254 radius=0.105
- link wheel_3/J1_base/INPUT_INTERFACE: geometry collision cylinder length=0.025 radius=0.035; visual cylinder length=0.025 radius=0.035
- link wheel_3/J2_shoulder/INPUT_INTERFACE: geometry collision cylinder length=0.04 radius=0.035; visual cylinder length=0.04 radius=0.035
- link wheel_3/wheel/INPUT_INTERFACE: geometry collision cylinder length=0.0254 radius=0.105; visual cylinder length=0.0254 radius=0.105
- link wheel_4/J1_base/INPUT_INTERFACE: geometry collision cylinder length=0.025 radius=0.035; visual cylinder length=0.025 radius=0.035
- link wheel_4/J2_shoulder/INPUT_INTERFACE: geometry collision cylinder length=0.04 radius=0.035; visual cylinder length=0.04 radius=0.035
- link wheel_4/wheel/INPUT_INTERFACE: geometry collision cylinder length=0.0254 radius=0.105; visual cylinder length=0.0254 radius=0.105
- link wheel_5/J1_base/INPUT_INTERFACE: geometry collision cylinder length=0.025 radius=0.035; visual cylinder length=0.025 radius=0.035
- link wheel_5/J2_shoulder/INPUT_INTERFACE: geometry collision cylinder length=0.04 radius=0.035; visual cylinder length=0.04 radius=0.035
- link wheel_5/wheel/INPUT_INTERFACE: geometry collision cylinder length=0.0254 radius=0.105; visual cylinder length=0.0254 radius=0.105
- link wheel_6/J1_base/INPUT_INTERFACE: geometry collision cylinder length=0.025 radius=0.035; visual cylinder length=0.025 radius=0.035
- link wheel_6/J2_shoulder/INPUT_INTERFACE: geometry collision cylinder length=0.04 radius=0.035; visual cylinder length=0.04 radius=0.035
- link wheel_6/wheel/INPUT_INTERFACE: geometry collision cylinder length=0.0254 radius=0.105; visual cylinder length=0.0254 radius=0.105
