Commit message: before testing dummy controllers

File: urdf/actuator.xacro (robot description, xacro)
@@ -77,13 +77,13 @@
       <visual>
         <xacro:if value="${model_name.startswith('X5')}">
-          <origin xyz="0 0 0.0125" rpy="0 0 0" />
+        <origin xyz="0 0 0" rpy="0 0 0" />
           <geometry>
-            <cylinder radius="0.035" length="0.025"/>
+            <mesh filename="${mesh_filename}" scale="0.001 0.001 0.001"/>
           </geometry>
         </xacro:if>
         <xacro:if value="${model_name.startswith('X8')}">
-          <origin xyz="0 0 0.02" rpy="0 0 0" />
+        <origin xyz="0 0 0" rpy="0 0 0" />
           <geometry>
-            <cylinder radius="0.035" length="0.04"/>
+            <mesh filename="${mesh_filename}" scale="0.001 0.001 0.001"/>
           </geometry>
         </xacro:if>

File: urdf/bracket.xacro (robot description, xacro)
@@ -49,5 +49,4 @@
     <!-- Heavy bracket -->
     <xacro:if value="${bracket_type.startswith('X5Heavy') or bracket_type.startswith('R5Heavy')}">
-      <!-- REMOVED VISUAL AND COLLISION FOR SPEED
       <visual>
         <xacro:if value="${bracket_type.endswith('RightOutside')}">
@@ -91,4 +90,5 @@
         <xacro:black_material/>
       </visual>
+      <!-- REMOVED COLLISION FOR SPEED
       <collision>
         <xacro:if value="${bracket_type.endswith('RightOutside')}">

File: urdf/llllll.urdf (robot description, URDF)
Before this commit: robot llllll, 43 links, 42 joints
Links:
- link leg_1/J1_base/INPUT_INTERFACE: geometry collision cylinder length=0.04 radius=0.035; visual mesh filename=X8.stl scale=0.001 0.001 0.001
- link leg_1/J2_shoulder/INPUT_INTERFACE: geometry collision cylinder length=0.04 radius=0.035; visual mesh filename=X8.stl scale=0.001 0.001 0.001
- link leg_1/J3_elbow/INPUT_INTERFACE: geometry collision cylinder length=0.025 radius=0.035; visual mesh filename=X5.stl scale=0.001 0.001 0.001
- link leg_1/shoulder_bracket/INPUT_INTERFACE: geometry visual mesh filename=PM-2149-01.stl scale=0.001 0.001 0.001; visual mesh filename=PM-2150-01R.stl scale=0.001 0.001 0.001
- link leg_2/J1_base/INPUT_INTERFACE: geometry collision cylinder length=0.04 radius=0.035; visual mesh filename=X8.stl scale=0.001 0.001 0.001
- link leg_2/J2_shoulder/INPUT_INTERFACE: geometry collision cylinder length=0.04 radius=0.035; visual mesh filename=X8.stl scale=0.001 0.001 0.001
- link leg_2/J3_elbow/INPUT_INTERFACE: geometry collision cylinder length=0.025 radius=0.035; visual mesh filename=X5.stl scale=0.001 0.001 0.001
- link leg_2/shoulder_bracket/INPUT_INTERFACE: geometry visual mesh filename=PM-2149-01.stl scale=0.001 0.001 0.001; visual mesh filename=PM-2150-01R.stl scale=0.001 0.001 0.001
- link leg_3/J1_base/INPUT_INTERFACE: geometry collision cylinder length=0.04 radius=0.035; visual mesh filename=X8.stl scale=0.001 0.001 0.001
- link leg_3/J2_shoulder/INPUT_INTERFACE: geometry collision cylinder length=0.04 radius=0.035; visual mesh filename=X8.stl scale=0.001 0.001 0.001
- link leg_3/J3_elbow/INPUT_INTERFACE: geometry collision cylinder length=0.025 radius=0.035; visual mesh filename=X5.stl scale=0.001 0.001 0.001
- link leg_3/shoulder_bracket/INPUT_INTERFACE: geometry visual mesh filename=PM-2149-01.stl scale=0.001 0.001 0.001; visual mesh filename=PM-2150-01R.stl scale=0.001 0.001 0.001
- link leg_4/J1_base/INPUT_INTERFACE: geometry collision cylinder length=0.04 radius=0.035; visual mesh filename=X8.stl scale=0.001 0.001 0.001
- link leg_4/J2_shoulder/INPUT_INTERFACE: geometry collision cylinder length=0.04 radius=0.035; visual mesh filename=X8.stl scale=0.001 0.001 0.001
- link leg_4/J3_elbow/INPUT_INTERFACE: geometry collision cylinder length=0.025 radius=0.035; visual mesh filename=X5.stl scale=0.001 0.001 0.001
- link leg_4/shoulder_bracket/INPUT_INTERFACE: geometry visual mesh filename=PM-2149-01.stl scale=0.001 0.001 0.001; visual mesh filename=PM-2150-01R.stl scale=0.001 0.001 0.001
- link leg_5/J1_base/INPUT_INTERFACE: geometry collision cylinder length=0.04 radius=0.035; visual mesh filename=X8.stl scale=0.001 0.001 0.001
- link leg_5/J2_shoulder/INPUT_INTERFACE: geometry collision cylinder length=0.04 radius=0.035; visual mesh filename=X8.stl scale=0.001 0.001 0.001
- link leg_5/J3_elbow/INPUT_INTERFACE: geometry collision cylinder length=0.025 radius=0.035; visual mesh filename=X5.stl scale=0.001 0.001 0.001
- link leg_5/shoulder_bracket/INPUT_INTERFACE: geometry visual mesh filename=PM-2149-01.stl scale=0.001 0.001 0.001; visual mesh filename=PM-2150-01R.stl scale=0.001 0.001 0.001
- link leg_6/J1_base/INPUT_INTERFACE: geometry collision cylinder length=0.04 radius=0.035; visual mesh filename=X8.stl scale=0.001 0.001 0.001
- link leg_6/J2_shoulder/INPUT_INTERFACE: geometry collision cylinder length=0.04 radius=0.035; visual mesh filename=X8.stl scale=0.001 0.001 0.001
- link leg_6/J3_elbow/INPUT_INTERFACE: geometry collision cylinder length=0.025 radius=0.035; visual mesh filename=X5.stl scale=0.001 0.001 0.001
- link leg_6/shoulder_bracket/INPUT_INTERFACE: geometry visual mesh filename=PM-2149-01.stl scale=0.001 0.001 0.001; visual mesh filename=PM-2150-01R.stl scale=0.001 0.001 0.001

File: urdf/llllll.xacro (robot description, xacro)
@@ -4,4 +4,5 @@
 <xacro:include filename="leg.xacro"/>
 <xacro:include filename="wheel.xacro"/>
+<xacro:include filename="wheelleg.xacro"/>
 <xacro:include filename="chassis.xacro"/>
 <xacro:chassis/>

File: urdf/llwwll.urdf (robot description, URDF)
Before this commit: robot llwwll, 37 links, 36 joints
Links:
- link leg_1/J1_base/INPUT_INTERFACE: geometry collision cylinder length=0.04 radius=0.035; visual mesh filename=X8.stl scale=0.001 0.001 0.001
- link leg_1/J2_shoulder/INPUT_INTERFACE: geometry collision cylinder length=0.04 radius=0.035; visual mesh filename=X8.stl scale=0.001 0.001 0.001
- link leg_1/J3_elbow/INPUT_INTERFACE: geometry collision cylinder length=0.025 radius=0.035; visual mesh filename=X5.stl scale=0.001 0.001 0.001
- link leg_1/shoulder_bracket/INPUT_INTERFACE: geometry visual mesh filename=PM-2149-01.stl scale=0.001 0.001 0.001; visual mesh filename=PM-2150-01R.stl scale=0.001 0.001 0.001
- link leg_2/J1_base/INPUT_INTERFACE: geometry collision cylinder length=0.04 radius=0.035; visual mesh filename=X8.stl scale=0.001 0.001 0.001
- link leg_2/J2_shoulder/INPUT_INTERFACE: geometry collision cylinder length=0.04 radius=0.035; visual mesh filename=X8.stl scale=0.001 0.001 0.001
- link leg_2/J3_elbow/INPUT_INTERFACE: geometry collision cylinder length=0.025 radius=0.035; visual mesh filename=X5.stl scale=0.001 0.001 0.001
- link leg_2/shoulder_bracket/INPUT_INTERFACE: geometry visual mesh filename=PM-2149-01.stl scale=0.001 0.001 0.001; visual mesh filename=PM-2150-01R.stl scale=0.001 0.001 0.001
- link leg_5/J1_base/INPUT_INTERFACE: geometry collision cylinder length=0.04 radius=0.035; visual mesh filename=X8.stl scale=0.001 0.001 0.001
- link leg_5/J2_shoulder/INPUT_INTERFACE: geometry collision cylinder length=0.04 radius=0.035; visual mesh filename=X8.stl scale=0.001 0.001 0.001
- link leg_5/J3_elbow/INPUT_INTERFACE: geometry collision cylinder length=0.025 radius=0.035; visual mesh filename=X5.stl scale=0.001 0.001 0.001
- link leg_5/shoulder_bracket/INPUT_INTERFACE: geometry visual mesh filename=PM-2149-01.stl scale=0.001 0.001 0.001; visual mesh filename=PM-2150-01R.stl scale=0.001 0.001 0.001
- link leg_6/J1_base/INPUT_INTERFACE: geometry collision cylinder length=0.04 radius=0.035; visual mesh filename=X8.stl scale=0.001 0.001 0.001
- link leg_6/J2_shoulder/INPUT_INTERFACE: geometry collision cylinder length=0.04 radius=0.035; visual mesh filename=X8.stl scale=0.001 0.001 0.001
- link leg_6/J3_elbow/INPUT_INTERFACE: geometry collision cylinder length=0.025 radius=0.035; visual mesh filename=X5.stl scale=0.001 0.001 0.001
- link leg_6/shoulder_bracket/INPUT_INTERFACE: geometry visual mesh filename=PM-2149-01.stl scale=0.001 0.001 0.001; visual mesh filename=PM-2150-01R.stl scale=0.001 0.001 0.001
- link wheel_3/J1_base/INPUT_INTERFACE: geometry collision cylinder length=0.025 radius=0.035; visual mesh filename=X5.stl scale=0.001 0.001 0.001
- link wheel_3/J2_shoulder/INPUT_INTERFACE: mass 0.48 -> 0.46; geometry collision cylinder length=0.04 radius=0.035; visual mesh filename=X8.stl scale=0.001 0.001 0.001
- link wheel_3/shoulder_bracket/INPUT_INTERFACE: geometry visual mesh filename=PM-2149-01.stl scale=0.001 0.001 0.001; visual mesh filename=PM-2150-01R.stl scale=0.001 0.001 0.001
- link wheel_4/J1_base/INPUT_INTERFACE: geometry collision cylinder length=0.025 radius=0.035; visual mesh filename=X5.stl scale=0.001 0.001 0.001
- link wheel_4/J2_shoulder/INPUT_INTERFACE: mass 0.48 -> 0.46; geometry collision cylinder length=0.04 radius=0.035; visual mesh filename=X8.stl scale=0.001 0.001 0.001
- link wheel_4/shoulder_bracket/INPUT_INTERFACE: geometry visual mesh filename=PM-2149-01.stl scale=0.001 0.001 0.001; visual mesh filename=PM-2150-01R.stl scale=0.001 0.001 0.001
Joints:
- removed joint wheel_3/J2_shoulder/X8_9
- removed joint wheel_4/J2_shoulder/X8_9
- added joint wheel_3/J2_shoulder/X8_3: type continuous, parent wheel_3/J2_shoulder/INPUT_INTERFACE, child wheel_3/wheel/INPUT_INTERFACE, origin xyz=0 0 0.045 rpy=0 0 0, axis 0 0 1, limit effort=7 velocity=8.796
- added joint wheel_4/J2_shoulder/X8_3: type continuous, parent wheel_4/J2_shoulder/INPUT_INTERFACE, child wheel_4/wheel/INPUT_INTERFACE, origin xyz=0 0 0.045 rpy=0 0 0, axis 0 0 1, limit effort=7 velocity=8.796

File: urdf/llwwll.xacro (robot description, xacro)
@@ -4,4 +4,5 @@
 <xacro:include filename="leg.xacro"/>
 <xacro:include filename="wheel.xacro"/>
+<xacro:include filename="wheelleg.xacro"/>
 <xacro:include filename="chassis.xacro"/>
 <xacro:chassis/>

File: urdf/lnllnl.urdf (robot description, URDF)
Before this commit: robot lnllnl, 29 links, 28 joints
Links:
- link leg_1/J1_base/INPUT_INTERFACE: geometry collision cylinder length=0.04 radius=0.035; visual mesh filename=X8.stl scale=0.001 0.001 0.001
- link leg_1/J2_shoulder/INPUT_INTERFACE: geometry collision cylinder length=0.04 radius=0.035; visual mesh filename=X8.stl scale=0.001 0.001 0.001
- link leg_1/J3_elbow/INPUT_INTERFACE: geometry collision cylinder length=0.025 radius=0.035; visual mesh filename=X5.stl scale=0.001 0.001 0.001
- link leg_1/shoulder_bracket/INPUT_INTERFACE: geometry visual mesh filename=PM-2149-01.stl scale=0.001 0.001 0.001; visual mesh filename=PM-2150-01R.stl scale=0.001 0.001 0.001
- link leg_3/J1_base/INPUT_INTERFACE: geometry collision cylinder length=0.04 radius=0.035; visual mesh filename=X8.stl scale=0.001 0.001 0.001
- link leg_3/J2_shoulder/INPUT_INTERFACE: geometry collision cylinder length=0.04 radius=0.035; visual mesh filename=X8.stl scale=0.001 0.001 0.001
- link leg_3/J3_elbow/INPUT_INTERFACE: geometry collision cylinder length=0.025 radius=0.035; visual mesh filename=X5.stl scale=0.001 0.001 0.001
- link leg_3/shoulder_bracket/INPUT_INTERFACE: geometry visual mesh filename=PM-2149-01.stl scale=0.001 0.001 0.001; visual mesh filename=PM-2150-01R.stl scale=0.001 0.001 0.001
- link leg_4/J1_base/INPUT_INTERFACE: geometry collision cylinder length=0.04 radius=0.035; visual mesh filename=X8.stl scale=0.001 0.001 0.001
- link leg_4/J2_shoulder/INPUT_INTERFACE: geometry collision cylinder length=0.04 radius=0.035; visual mesh filename=X8.stl scale=0.001 0.001 0.001
- link leg_4/J3_elbow/INPUT_INTERFACE: geometry collision cylinder length=0.025 radius=0.035; visual mesh filename=X5.stl scale=0.001 0.001 0.001
- link leg_4/shoulder_bracket/INPUT_INTERFACE: geometry visual mesh filename=PM-2149-01.stl scale=0.001 0.001 0.001; visual mesh filename=PM-2150-01R.stl scale=0.001 0.001 0.001
- link leg_6/J1_base/INPUT_INTERFACE: geometry collision cylinder length=0.04 radius=0.035; visual mesh filename=X8.stl scale=0.001 0.001 0.001
- link leg_6/J2_shoulder/INPUT_INTERFACE: geometry collision cylinder length=0.04 radius=0.035; visual mesh filename=X8.stl scale=0.001 0.001 0.001
- link leg_6/J3_elbow/INPUT_INTERFACE: geometry collision cylinder length=0.025 radius=0.035; visual mesh filename=X5.stl scale=0.001 0.001 0.001
- link leg_6/shoulder_bracket/INPUT_INTERFACE: geometry visual mesh filename=PM-2149-01.stl scale=0.001 0.001 0.001; visual mesh filename=PM-2150-01R.stl scale=0.001 0.001 0.001

File: urdf/lnllnl.xacro (robot description, xacro)
@@ -4,4 +4,5 @@
 <xacro:include filename="leg.xacro"/>
 <xacro:include filename="wheel.xacro"/>
+<xacro:include filename="wheelleg.xacro"/>
 <xacro:include filename="chassis.xacro"/>
 <xacro:chassis/>

File: urdf/lnwwnl.urdf (robot description, URDF)
Before this commit: robot lnwwnl, 23 links, 22 joints
Links:
- link leg_1/J1_base/INPUT_INTERFACE: geometry collision cylinder length=0.04 radius=0.035; visual mesh filename=X8.stl scale=0.001 0.001 0.001
- link leg_1/J2_shoulder/INPUT_INTERFACE: geometry collision cylinder length=0.04 radius=0.035; visual mesh filename=X8.stl scale=0.001 0.001 0.001
- link leg_1/J3_elbow/INPUT_INTERFACE: geometry collision cylinder length=0.025 radius=0.035; visual mesh filename=X5.stl scale=0.001 0.001 0.001
- link leg_1/shoulder_bracket/INPUT_INTERFACE: geometry visual mesh filename=PM-2149-01.stl scale=0.001 0.001 0.001; visual mesh filename=PM-2150-01R.stl scale=0.001 0.001 0.001
- link leg_6/J1_base/INPUT_INTERFACE: geometry collision cylinder length=0.04 radius=0.035; visual mesh filename=X8.stl scale=0.001 0.001 0.001
- link leg_6/J2_shoulder/INPUT_INTERFACE: geometry collision cylinder length=0.04 radius=0.035; visual mesh filename=X8.stl scale=0.001 0.001 0.001
- link leg_6/J3_elbow/INPUT_INTERFACE: geometry collision cylinder length=0.025 radius=0.035; visual mesh filename=X5.stl scale=0.001 0.001 0.001
- link leg_6/shoulder_bracket/INPUT_INTERFACE: geometry visual mesh filename=PM-2149-01.stl scale=0.001 0.001 0.001; visual mesh filename=PM-2150-01R.stl scale=0.001 0.001 0.001
- link wheel_3/J1_base/INPUT_INTERFACE: geometry collision cylinder length=0.025 radius=0.035; visual mesh filename=X5.stl scale=0.001 0.001 0.001
- link wheel_3/J2_shoulder/INPUT_INTERFACE: mass 0.48 -> 0.46; geometry collision cylinder length=0.04 radius=0.035; visual mesh filename=X8.stl scale=0.001 0.001 0.001
- link wheel_3/shoulder_bracket/INPUT_INTERFACE: geometry visual mesh filename=PM-2149-01.stl scale=0.001 0.001 0.001; visual mesh filename=PM-2150-01R.stl scale=0.001 0.001 0.001
- link wheel_4/J1_base/INPUT_INTERFACE: geometry collision cylinder length=0.025 radius=0.035; visual mesh filename=X5.stl scale=0.001 0.001 0.001
- link wheel_4/J2_shoulder/INPUT_INTERFACE: mass 0.48 -> 0.46; geometry collision cylinder length=0.04 radius=0.035; visual mesh filename=X8.stl scale=0.001 0.001 0.001
- link wheel_4/shoulder_bracket/INPUT_INTERFACE: geometry visual mesh filename=PM-2149-01.stl scale=0.001 0.001 0.001; visual mesh filename=PM-2150-01R.stl scale=0.001 0.001 0.001
Joints:
- removed joint wheel_3/J2_shoulder/X8_9
- removed joint wheel_4/J2_shoulder/X8_9
- added joint wheel_3/J2_shoulder/X8_3: type continuous, parent wheel_3/J2_shoulder/INPUT_INTERFACE, child wheel_3/wheel/INPUT_INTERFACE, origin xyz=0 0 0.045 rpy=0 0 0, axis 0 0 1, limit effort=7 velocity=8.796
- added joint wheel_4/J2_shoulder/X8_3: type continuous, parent wheel_4/J2_shoulder/INPUT_INTERFACE, child wheel_4/wheel/INPUT_INTERFACE, origin xyz=0 0 0.045 rpy=0 0 0, axis 0 0 1, limit effort=7 velocity=8.796

File: urdf/lnwwnl.xacro (robot description, xacro)
@@ -4,4 +4,5 @@
 <xacro:include filename="leg.xacro"/>
 <xacro:include filename="wheel.xacro"/>
+<xacro:include filename="wheelleg.xacro"/>
 <xacro:include filename="chassis.xacro"/>
 <xacro:chassis/>

File: urdf/lwllwl.urdf (robot description, URDF)
Before this commit: robot lwllwl, 37 links, 36 joints
Links:
- link leg_1/J1_base/INPUT_INTERFACE: geometry collision cylinder length=0.04 radius=0.035; visual mesh filename=X8.stl scale=0.001 0.001 0.001
- link leg_1/J2_shoulder/INPUT_INTERFACE: geometry collision cylinder length=0.04 radius=0.035; visual mesh filename=X8.stl scale=0.001 0.001 0.001
- link leg_1/J3_elbow/INPUT_INTERFACE: geometry collision cylinder length=0.025 radius=0.035; visual mesh filename=X5.stl scale=0.001 0.001 0.001
- link leg_1/shoulder_bracket/INPUT_INTERFACE: geometry visual mesh filename=PM-2149-01.stl scale=0.001 0.001 0.001; visual mesh filename=PM-2150-01R.stl scale=0.001 0.001 0.001
- link leg_3/J1_base/INPUT_INTERFACE: geometry collision cylinder length=0.04 radius=0.035; visual mesh filename=X8.stl scale=0.001 0.001 0.001
- link leg_3/J2_shoulder/INPUT_INTERFACE: geometry collision cylinder length=0.04 radius=0.035; visual mesh filename=X8.stl scale=0.001 0.001 0.001
- link leg_3/J3_elbow/INPUT_INTERFACE: geometry collision cylinder length=0.025 radius=0.035; visual mesh filename=X5.stl scale=0.001 0.001 0.001
- link leg_3/shoulder_bracket/INPUT_INTERFACE: geometry visual mesh filename=PM-2149-01.stl scale=0.001 0.001 0.001; visual mesh filename=PM-2150-01R.stl scale=0.001 0.001 0.001
- link leg_4/J1_base/INPUT_INTERFACE: geometry collision cylinder length=0.04 radius=0.035; visual mesh filename=X8.stl scale=0.001 0.001 0.001
- link leg_4/J2_shoulder/INPUT_INTERFACE: geometry collision cylinder length=0.04 radius=0.035; visual mesh filename=X8.stl scale=0.001 0.001 0.001
- link leg_4/J3_elbow/INPUT_INTERFACE: geometry collision cylinder length=0.025 radius=0.035; visual mesh filename=X5.stl scale=0.001 0.001 0.001
- link leg_4/shoulder_bracket/INPUT_INTERFACE: geometry visual mesh filename=PM-2149-01.stl scale=0.001 0.001 0.001; visual mesh filename=PM-2150-01R.stl scale=0.001 0.001 0.001
- link leg_6/J1_base/INPUT_INTERFACE: geometry collision cylinder length=0.04 radius=0.035; visual mesh filename=X8.stl scale=0.001 0.001 0.001
- link leg_6/J2_shoulder/INPUT_INTERFACE: geometry collision cylinder length=0.04 radius=0.035; visual mesh filename=X8.stl scale=0.001 0.001 0.001
- link leg_6/J3_elbow/INPUT_INTERFACE: geometry collision cylinder length=0.025 radius=0.035; visual mesh filename=X5.stl scale=0.001 0.001 0.001
- link leg_6/shoulder_bracket/INPUT_INTERFACE: geometry visual mesh filename=PM-2149-01.stl scale=0.001 0.001 0.001; visual mesh filename=PM-2150-01R.stl scale=0.001 0.001 0.001
- link wheel_2/J1_base/INPUT_INTERFACE: geometry collision cylinder length=0.025 radius=0.035; visual mesh filename=X5.stl scale=0.001 0.001 0.001
- link wheel_2/J2_shoulder/INPUT_INTERFACE: mass 0.48 -> 0.46; geometry collision cylinder length=0.04 radius=0.035; visual mesh filename=X8.stl scale=0.001 0.001 0.001
- link wheel_2/shoulder_bracket/INPUT_INTERFACE: geometry visual mesh filename=PM-2149-01.stl scale=0.001 0.001 0.001; visual mesh filename=PM-2150-01R.stl scale=0.001 0.001 0.001
- link wheel_5/J1_base/INPUT_INTERFACE: geometry collision cylinder length=0.025 radius=0.035; visual mesh filename=X5.stl scale=0.001 0.001 0.001
- link wheel_5/J2_shoulder/INPUT_INTERFACE: mass 0.48 -> 0.46; geometry collision cylinder length=0.04 radius=0.035; visual mesh filename=X8.stl scale=0.001 0.001 0.001
- link wheel_5/shoulder_bracket/INPUT_INTERFACE: geometry visual mesh filename=PM-2149-01.stl scale=0.001 0.001 0.001; visual mesh filename=PM-2150-01R.stl scale=0.001 0.001 0.001
Joints:
- removed joint wheel_2/J2_shoulder/X8_9
- removed joint wheel_5/J2_shoulder/X8_9
- added joint wheel_2/J2_shoulder/X8_3: type continuous, parent wheel_2/J2_shoulder/INPUT_INTERFACE, child wheel_2/wheel/INPUT_INTERFACE, origin xyz=0 0 0.045 rpy=0 0 0, axis 0 0 1, limit effort=7 velocity=8.796
- added joint wheel_5/J2_shoulder/X8_3: type continuous, parent wheel_5/J2_shoulder/INPUT_INTERFACE, child wheel_5/wheel/INPUT_INTERFACE, origin xyz=0 0 0.045 rpy=0 0 0, axis 0 0 1, limit effort=7 velocity=8.796

File: urdf/lwllwl.xacro (robot description, xacro)
@@ -4,4 +4,5 @@
 <xacro:include filename="leg.xacro"/>
 <xacro:include filename="wheel.xacro"/>
+<xacro:include filename="wheelleg.xacro"/>
 <xacro:include filename="chassis.xacro"/>
 <xacro:chassis/>
