Commit message: before testing dummy controllers

File: urdf/lwwwwl.urdf (robot description, URDF)
Before this commit: robot lwwwwl, 31 links, 30 joints
Links:
- link leg_1/J1_base/INPUT_INTERFACE: geometry collision cylinder length=0.04 radius=0.035; visual mesh filename=X8.stl scale=0.001 0.001 0.001
- link leg_1/J2_shoulder/INPUT_INTERFACE: geometry collision cylinder length=0.04 radius=0.035; visual mesh filename=X8.stl scale=0.001 0.001 0.001
- link leg_1/J3_elbow/INPUT_INTERFACE: geometry collision cylinder length=0.025 radius=0.035; visual mesh filename=X5.stl scale=0.001 0.001 0.001
- link leg_1/shoulder_bracket/INPUT_INTERFACE: geometry visual mesh filename=PM-2149-01.stl scale=0.001 0.001 0.001; visual mesh filename=PM-2150-01R.stl scale=0.001 0.001 0.001
- link leg_6/J1_base/INPUT_INTERFACE: geometry collision cylinder length=0.04 radius=0.035; visual mesh filename=X8.stl scale=0.001 0.001 0.001
- link leg_6/J2_shoulder/INPUT_INTERFACE: geometry collision cylinder length=0.04 radius=0.035; visual mesh filename=X8.stl scale=0.001 0.001 0.001
- link leg_6/J3_elbow/INPUT_INTERFACE: geometry collision cylinder length=0.025 radius=0.035; visual mesh filename=X5.stl scale=0.001 0.001 0.001
- link leg_6/shoulder_bracket/INPUT_INTERFACE: geometry visual mesh filename=PM-2149-01.stl scale=0.001 0.001 0.001; visual mesh filename=PM-2150-01R.stl scale=0.001 0.001 0.001
- link wheel_2/J1_base/INPUT_INTERFACE: geometry collision cylinder length=0.025 radius=0.035; visual mesh filename=X5.stl scale=0.001 0.001 0.001
- link wheel_2/J2_shoulder/INPUT_INTERFACE: mass 0.48 -> 0.46; geometry collision cylinder length=0.04 radius=0.035; visual mesh filename=X8.stl scale=0.001 0.001 0.001
- link wheel_2/shoulder_bracket/INPUT_INTERFACE: geometry visual mesh filename=PM-2149-01.stl scale=0.001 0.001 0.001; visual mesh filename=PM-2150-01R.stl scale=0.001 0.001 0.001
- link wheel_3/J1_base/INPUT_INTERFACE: geometry collision cylinder length=0.025 radius=0.035; visual mesh filename=X5.stl scale=0.001 0.001 0.001
- link wheel_3/J2_shoulder/INPUT_INTERFACE: mass 0.48 -> 0.46; geometry collision cylinder length=0.04 radius=0.035; visual mesh filename=X8.stl scale=0.001 0.001 0.001
- link wheel_3/shoulder_bracket/INPUT_INTERFACE: geometry visual mesh filename=PM-2149-01.stl scale=0.001 0.001 0.001; visual mesh filename=PM-2150-01R.stl scale=0.001 0.001 0.001
- link wheel_4/J1_base/INPUT_INTERFACE: geometry collision cylinder length=0.025 radius=0.035; visual mesh filename=X5.stl scale=0.001 0.001 0.001
- link wheel_4/J2_shoulder/INPUT_INTERFACE: mass 0.48 -> 0.46; geometry collision cylinder length=0.04 radius=0.035; visual mesh filename=X8.stl scale=0.001 0.001 0.001
- link wheel_4/shoulder_bracket/INPUT_INTERFACE: geometry visual mesh filename=PM-2149-01.stl scale=0.001 0.001 0.001; visual mesh filename=PM-2150-01R.stl scale=0.001 0.001 0.001
- link wheel_5/J1_base/INPUT_INTERFACE: geometry collision cylinder length=0.025 radius=0.035; visual mesh filename=X5.stl scale=0.001 0.001 0.001
- link wheel_5/J2_shoulder/INPUT_INTERFACE: mass 0.48 -> 0.46; geometry collision cylinder length=0.04 radius=0.035; visual mesh filename=X8.stl scale=0.001 0.001 0.001
- link wheel_5/shoulder_bracket/INPUT_INTERFACE: geometry visual mesh filename=PM-2149-01.stl scale=0.001 0.001 0.001; visual mesh filename=PM-2150-01R.stl scale=0.001 0.001 0.001
Joints:
- removed joint wheel_2/J2_shoulder/X8_9
- removed joint wheel_3/J2_shoulder/X8_9
- removed joint wheel_4/J2_shoulder/X8_9
- removed joint wheel_5/J2_shoulder/X8_9
- added joint wheel_2/J2_shoulder/X8_3: type continuous, parent wheel_2/J2_shoulder/INPUT_INTERFACE, child wheel_2/wheel/INPUT_INTERFACE, origin xyz=0 0 0.045 rpy=0 0 0, axis 0 0 1, limit effort=7 velocity=8.796
- added joint wheel_3/J2_shoulder/X8_3: type continuous, parent wheel_3/J2_shoulder/INPUT_INTERFACE, child wheel_3/wheel/INPUT_INTERFACE, origin xyz=0 0 0.045 rpy=0 0 0, axis 0 0 1, limit effort=7 velocity=8.796
- added joint wheel_4/J2_shoulder/X8_3: type continuous, parent wheel_4/J2_shoulder/INPUT_INTERFACE, child wheel_4/wheel/INPUT_INTERFACE, origin xyz=0 0 0.045 rpy=0 0 0, axis 0 0 1, limit effort=7 velocity=8.796
- added joint wheel_5/J2_shoulder/X8_3: type continuous, parent wheel_5/J2_shoulder/INPUT_INTERFACE, child wheel_5/wheel/INPUT_INTERFACE, origin xyz=0 0 0.045 rpy=0 0 0, axis 0 0 1, limit effort=7 velocity=8.796

File: urdf/lwwwwl.xacro (robot description, xacro)
@@ -4,4 +4,5 @@
 <xacro:include filename="leg.xacro"/>
 <xacro:include filename="wheel.xacro"/>
+<xacro:include filename="wheelleg.xacro"/>
 <xacro:include filename="chassis.xacro"/>
 <xacro:chassis/>

File: urdf/wheel.xacro (robot description, xacro)
@@ -10,5 +10,5 @@
 <xacro:actuator name="wheel_${num}/J1_base" child="wheel_${num}/shoulder_bracket" type="X5_9" limits="${[-pi/3,pi/3]}"/>
 <xacro:bracket  name="wheel_${num}/shoulder_bracket" child="wheel_${num}/J2_shoulder" type="X5HeavyRightOutside"/>
-<xacro:actuator name="wheel_${num}/J2_shoulder" child="wheel_${num}/wheel" type="X8_9"/>
+<xacro:actuator name="wheel_${num}/J2_shoulder" child="wheel_${num}/wheel" type="X8_3"/>
   <link name="wheel_${num}/wheel/INPUT_INTERFACE">
     <inertial>

File: urdf/wllllw.urdf (robot description, URDF)
Before this commit: robot wllllw, 37 links, 36 joints
Links:
- link leg_2/J1_base/INPUT_INTERFACE: geometry collision cylinder length=0.04 radius=0.035; visual mesh filename=X8.stl scale=0.001 0.001 0.001
- link leg_2/J2_shoulder/INPUT_INTERFACE: geometry collision cylinder length=0.04 radius=0.035; visual mesh filename=X8.stl scale=0.001 0.001 0.001
- link leg_2/J3_elbow/INPUT_INTERFACE: geometry collision cylinder length=0.025 radius=0.035; visual mesh filename=X5.stl scale=0.001 0.001 0.001
- link leg_2/shoulder_bracket/INPUT_INTERFACE: geometry visual mesh filename=PM-2149-01.stl scale=0.001 0.001 0.001; visual mesh filename=PM-2150-01R.stl scale=0.001 0.001 0.001
- link leg_3/J1_base/INPUT_INTERFACE: geometry collision cylinder length=0.04 radius=0.035; visual mesh filename=X8.stl scale=0.001 0.001 0.001
- link leg_3/J2_shoulder/INPUT_INTERFACE: geometry collision cylinder length=0.04 radius=0.035; visual mesh filename=X8.stl scale=0.001 0.001 0.001
- link leg_3/J3_elbow/INPUT_INTERFACE: geometry collision cylinder length=0.025 radius=0.035; visual mesh filename=X5.stl scale=0.001 0.001 0.001
- link leg_3/shoulder_bracket/INPUT_INTERFACE: geometry visual mesh filename=PM-2149-01.stl scale=0.001 0.001 0.001; visual mesh filename=PM-2150-01R.stl scale=0.001 0.001 0.001
- link leg_4/J1_base/INPUT_INTERFACE: geometry collision cylinder length=0.04 radius=0.035; visual mesh filename=X8.stl scale=0.001 0.001 0.001
- link leg_4/J2_shoulder/INPUT_INTERFACE: geometry collision cylinder length=0.04 radius=0.035; visual mesh filename=X8.stl scale=0.001 0.001 0.001
- link leg_4/J3_elbow/INPUT_INTERFACE: geometry collision cylinder length=0.025 radius=0.035; visual mesh filename=X5.stl scale=0.001 0.001 0.001
- link leg_4/shoulder_bracket/INPUT_INTERFACE: geometry visual mesh filename=PM-2149-01.stl scale=0.001 0.001 0.001; visual mesh filename=PM-2150-01R.stl scale=0.001 0.001 0.001
- link leg_5/J1_base/INPUT_INTERFACE: geometry collision cylinder length=0.04 radius=0.035; visual mesh filename=X8.stl scale=0.001 0.001 0.001
- link leg_5/J2_shoulder/INPUT_INTERFACE: geometry collision cylinder length=0.04 radius=0.035; visual mesh filename=X8.stl scale=0.001 0.001 0.001
- link leg_5/J3_elbow/INPUT_INTERFACE: geometry collision cylinder length=0.025 radius=0.035; visual mesh filename=X5.stl scale=0.001 0.001 0.001
- link leg_5/shoulder_bracket/INPUT_INTERFACE: geometry visual mesh filename=PM-2149-01.stl scale=0.001 0.001 0.001; visual mesh filename=PM-2150-01R.stl scale=0.001 0.001 0.001
- link wheel_1/J1_base/INPUT_INTERFACE: geometry collision cylinder length=0.025 radius=0.035; visual mesh filename=X5.stl scale=0.001 0.001 0.001
- link wheel_1/J2_shoulder/INPUT_INTERFACE: mass 0.48 -> 0.46; geometry collision cylinder length=0.04 radius=0.035; visual mesh filename=X8.stl scale=0.001 0.001 0.001
- link wheel_1/shoulder_bracket/INPUT_INTERFACE: geometry visual mesh filename=PM-2149-01.stl scale=0.001 0.001 0.001; visual mesh filename=PM-2150-01R.stl scale=0.001 0.001 0.001
- link wheel_6/J1_base/INPUT_INTERFACE: geometry collision cylinder length=0.025 radius=0.035; visual mesh filename=X5.stl scale=0.001 0.001 0.001
- link wheel_6/J2_shoulder/INPUT_INTERFACE: mass 0.48 -> 0.46; geometry collision cylinder length=0.04 radius=0.035; visual mesh filename=X8.stl scale=0.001 0.001 0.001
- link wheel_6/shoulder_bracket/INPUT_INTERFACE: geometry visual mesh filename=PM-2149-01.stl scale=0.001 0.001 0.001; visual mesh filename=PM-2150-01R.stl scale=0.001 0.001 0.001
Joints:
- removed joint wheel_1/J2_shoulder/X8_9
- removed joint wheel_6/J2_shoulder/X8_9
- added joint wheel_1/J2_shoulder/X8_3: type continuous, parent wheel_1/J2_shoulder/INPUT_INTERFACE, child wheel_1/wheel/INPUT_INTERFACE, origin xyz=0 0 0.045 rpy=0 0 0, axis 0 0 1, limit effort=7 velocity=8.796
- added joint wheel_6/J2_shoulder/X8_3: type continuous, parent wheel_6/J2_shoulder/INPUT_INTERFACE, child wheel_6/wheel/INPUT_INTERFACE, origin xyz=0 0 0.045 rpy=0 0 0, axis 0 0 1, limit effort=7 velocity=8.796

File: urdf/wllllw.xacro (robot description, xacro)
@@ -4,4 +4,5 @@
 <xacro:include filename="leg.xacro"/>
 <xacro:include filename="wheel.xacro"/>
+<xacro:include filename="wheelleg.xacro"/>
 <xacro:include filename="chassis.xacro"/>
 <xacro:chassis/>

File: urdf/wlwwlw.urdf (robot description, URDF)
Before this commit: robot wlwwlw, 31 links, 30 joints
Links:
- link leg_2/J1_base/INPUT_INTERFACE: geometry collision cylinder length=0.04 radius=0.035; visual mesh filename=X8.stl scale=0.001 0.001 0.001
- link leg_2/J2_shoulder/INPUT_INTERFACE: geometry collision cylinder length=0.04 radius=0.035; visual mesh filename=X8.stl scale=0.001 0.001 0.001
- link leg_2/J3_elbow/INPUT_INTERFACE: geometry collision cylinder length=0.025 radius=0.035; visual mesh filename=X5.stl scale=0.001 0.001 0.001
- link leg_2/shoulder_bracket/INPUT_INTERFACE: geometry visual mesh filename=PM-2149-01.stl scale=0.001 0.001 0.001; visual mesh filename=PM-2150-01R.stl scale=0.001 0.001 0.001
- link leg_5/J1_base/INPUT_INTERFACE: geometry collision cylinder length=0.04 radius=0.035; visual mesh filename=X8.stl scale=0.001 0.001 0.001
- link leg_5/J2_shoulder/INPUT_INTERFACE: geometry collision cylinder length=0.04 radius=0.035; visual mesh filename=X8.stl scale=0.001 0.001 0.001
- link leg_5/J3_elbow/INPUT_INTERFACE: geometry collision cylinder length=0.025 radius=0.035; visual mesh filename=X5.stl scale=0.001 0.001 0.001
- link leg_5/shoulder_bracket/INPUT_INTERFACE: geometry visual mesh filename=PM-2149-01.stl scale=0.001 0.001 0.001; visual mesh filename=PM-2150-01R.stl scale=0.001 0.001 0.001
- link wheel_1/J1_base/INPUT_INTERFACE: geometry collision cylinder length=0.025 radius=0.035; visual mesh filename=X5.stl scale=0.001 0.001 0.001
- link wheel_1/J2_shoulder/INPUT_INTERFACE: mass 0.48 -> 0.46; geometry collision cylinder length=0.04 radius=0.035; visual mesh filename=X8.stl scale=0.001 0.001 0.001
- link wheel_1/shoulder_bracket/INPUT_INTERFACE: geometry visual mesh filename=PM-2149-01.stl scale=0.001 0.001 0.001; visual mesh filename=PM-2150-01R.stl scale=0.001 0.001 0.001
- link wheel_3/J1_base/INPUT_INTERFACE: geometry collision cylinder length=0.025 radius=0.035; visual mesh filename=X5.stl scale=0.001 0.001 0.001
- link wheel_3/J2_shoulder/INPUT_INTERFACE: mass 0.48 -> 0.46; geometry collision cylinder length=0.04 radius=0.035; visual mesh filename=X8.stl scale=0.001 0.001 0.001
- link wheel_3/shoulder_bracket/INPUT_INTERFACE: geometry visual mesh filename=PM-2149-01.stl scale=0.001 0.001 0.001; visual mesh filename=PM-2150-01R.stl scale=0.001 0.001 0.001
- link wheel_4/J1_base/INPUT_INTERFACE: geometry collision cylinder length=0.025 radius=0.035; visual mesh filename=X5.stl scale=0.001 0.001 0.001
- link wheel_4/J2_shoulder/INPUT_INTERFACE: mass 0.48 -> 0.46; geometry collision cylinder length=0.04 radius=0.035; visual mesh filename=X8.stl scale=0.001 0.001 0.001
- link wheel_4/shoulder_bracket/INPUT_INTERFACE: geometry visual mesh filename=PM-2149-01.stl scale=0.001 0.001 0.001; visual mesh filename=PM-2150-01R.stl scale=0.001 0.001 0.001
- link wheel_6/J1_base/INPUT_INTERFACE: geometry collision cylinder length=0.025 radius=0.035; visual mesh filename=X5.stl scale=0.001 0.001 0.001
- link wheel_6/J2_shoulder/INPUT_INTERFACE: mass 0.48 -> 0.46; geometry collision cylinder length=0.04 radius=0.035; visual mesh filename=X8.stl scale=0.001 0.001 0.001
- link wheel_6/shoulder_bracket/INPUT_INTERFACE: geometry visual mesh filename=PM-2149-01.stl scale=0.001 0.001 0.001; visual mesh filename=PM-2150-01R.stl scale=0.001 0.001 0.001
Joints:
- removed joint wheel_1/J2_shoulder/X8_9
- removed joint wheel_3/J2_shoulder/X8_9
- removed joint wheel_4/J2_shoulder/X8_9
- removed joint wheel_6/J2_shoulder/X8_9
- added joint wheel_1/J2_shoulder/X8_3: type continuous, parent wheel_1/J2_shoulder/INPUT_INTERFACE, child wheel_1/wheel/INPUT_INTERFACE, origin xyz=0 0 0.045 rpy=0 0 0, axis 0 0 1, limit effort=7 velocity=8.796
- added joint wheel_3/J2_shoulder/X8_3: type continuous, parent wheel_3/J2_shoulder/INPUT_INTERFACE, child wheel_3/wheel/INPUT_INTERFACE, origin xyz=0 0 0.045 rpy=0 0 0, axis 0 0 1, limit effort=7 velocity=8.796
- added joint wheel_4/J2_shoulder/X8_3: type continuous, parent wheel_4/J2_shoulder/INPUT_INTERFACE, child wheel_4/wheel/INPUT_INTERFACE, origin xyz=0 0 0.045 rpy=0 0 0, axis 0 0 1, limit effort=7 velocity=8.796
- added joint wheel_6/J2_shoulder/X8_3: type continuous, parent wheel_6/J2_shoulder/INPUT_INTERFACE, child wheel_6/wheel/INPUT_INTERFACE, origin xyz=0 0 0.045 rpy=0 0 0, axis 0 0 1, limit effort=7 velocity=8.796

File: urdf/wlwwlw.xacro (robot description, xacro)
@@ -4,4 +4,5 @@
 <xacro:include filename="leg.xacro"/>
 <xacro:include filename="wheel.xacro"/>
+<xacro:include filename="wheelleg.xacro"/>
 <xacro:include filename="chassis.xacro"/>
 <xacro:chassis/>

File: urdf/wnllnw.urdf (robot description, URDF)
Before this commit: robot wnllnw, 23 links, 22 joints
Links:
- link leg_3/J1_base/INPUT_INTERFACE: geometry collision cylinder length=0.04 radius=0.035; visual mesh filename=X8.stl scale=0.001 0.001 0.001
- link leg_3/J2_shoulder/INPUT_INTERFACE: geometry collision cylinder length=0.04 radius=0.035; visual mesh filename=X8.stl scale=0.001 0.001 0.001
- link leg_3/J3_elbow/INPUT_INTERFACE: geometry collision cylinder length=0.025 radius=0.035; visual mesh filename=X5.stl scale=0.001 0.001 0.001
- link leg_3/shoulder_bracket/INPUT_INTERFACE: geometry visual mesh filename=PM-2149-01.stl scale=0.001 0.001 0.001; visual mesh filename=PM-2150-01R.stl scale=0.001 0.001 0.001
- link leg_4/J1_base/INPUT_INTERFACE: geometry collision cylinder length=0.04 radius=0.035; visual mesh filename=X8.stl scale=0.001 0.001 0.001
- link leg_4/J2_shoulder/INPUT_INTERFACE: geometry collision cylinder length=0.04 radius=0.035; visual mesh filename=X8.stl scale=0.001 0.001 0.001
- link leg_4/J3_elbow/INPUT_INTERFACE: geometry collision cylinder length=0.025 radius=0.035; visual mesh filename=X5.stl scale=0.001 0.001 0.001
- link leg_4/shoulder_bracket/INPUT_INTERFACE: geometry visual mesh filename=PM-2149-01.stl scale=0.001 0.001 0.001; visual mesh filename=PM-2150-01R.stl scale=0.001 0.001 0.001
- link wheel_1/J1_base/INPUT_INTERFACE: geometry collision cylinder length=0.025 radius=0.035; visual mesh filename=X5.stl scale=0.001 0.001 0.001
- link wheel_1/J2_shoulder/INPUT_INTERFACE: mass 0.48 -> 0.46; geometry collision cylinder length=0.04 radius=0.035; visual mesh filename=X8.stl scale=0.001 0.001 0.001
- link wheel_1/shoulder_bracket/INPUT_INTERFACE: geometry visual mesh filename=PM-2149-01.stl scale=0.001 0.001 0.001; visual mesh filename=PM-2150-01R.stl scale=0.001 0.001 0.001
- link wheel_6/J1_base/INPUT_INTERFACE: geometry collision cylinder length=0.025 radius=0.035; visual mesh filename=X5.stl scale=0.001 0.001 0.001
- link wheel_6/J2_shoulder/INPUT_INTERFACE: mass 0.48 -> 0.46; geometry collision cylinder length=0.04 radius=0.035; visual mesh filename=X8.stl scale=0.001 0.001 0.001
- link wheel_6/shoulder_bracket/INPUT_INTERFACE: geometry visual mesh filename=PM-2149-01.stl scale=0.001 0.001 0.001; visual mesh filename=PM-2150-01R.stl scale=0.001 0.001 0.001
Joints:
- removed joint wheel_1/J2_shoulder/X8_9
- removed joint wheel_6/J2_shoulder/X8_9
- added joint wheel_1/J2_shoulder/X8_3: type continuous, parent wheel_1/J2_shoulder/INPUT_INTERFACE, child wheel_1/wheel/INPUT_INTERFACE, origin xyz=0 0 0.045 rpy=0 0 0, axis 0 0 1, limit effort=7 velocity=8.796
- added joint wheel_6/J2_shoulder/X8_3: type continuous, parent wheel_6/J2_shoulder/INPUT_INTERFACE, child wheel_6/wheel/INPUT_INTERFACE, origin xyz=0 0 0.045 rpy=0 0 0, axis 0 0 1, limit effort=7 velocity=8.796
